File: pcb/hackpad-pcb.kicad_pcb (KiCad board)
At the start: 2 copper layers, 76.2 x 97.6 mm, 50 parts, among them J1 OLED_128x32, U1 MCU_Seeed_XIAO_RP2040

Commit message: Resized pcb and updated model
Signed-off-by: Urjith Mishra <66270347+TheScientist101@users.noreply.github.com>
Parts:
- moved D14 5.93 mm to (139.0, 132.0)
- moved D15 5.93 mm to (158.0, 132.0)
- moved D18 5.93 mm to (130.6, 76.0)
- moved D19 5.93 mm to (149.6, 76.0)
- moved D2 5.93 mm to (139.0, 74.9)
- moved D3 5.93 mm to (158.0, 74.9)
- moved D30 5.93 mm to (130.6, 133.2)
- moved D31 5.93 mm to (149.6, 133.2)
- moved D6 5.93 mm to (139.0, 93.9)
- moved D7 5.93 mm to (158.0, 93.9)
- moved S14 5.93 mm to (130.6, 128.1)
- moved S15 5.93 mm to (149.6, 128.1)
- moved S2 5.93 mm to (130.6, 71.0)
- moved S3 5.93 mm to (149.6, 71.0)
- moved S6 5.93 mm to (130.6, 90.0)
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Routing:
- net GND: track 354.8 -> 357.4 mm
- net +3V3: track 332.3 -> 331.2 mm
- net Row 0: track 95.6 -> 95.0 mm
Other:
- board size 76.2 x 97.6 mm -> 80 x 100 mm

Commit message: Add resistors for LEDs
Signed-off-by: Urjith Mishra <66270347+TheScientist101@users.noreply.github.com>
Parts:
- added R1: R, Resistor_THT:R_Axial_DIN0207_L6.3mm_D2.5mm_P7.62mm_Horizontal, B.Cu at (115.8, 62.0)
- added R10: R, Resistor_THT:R_Axial_DIN0207_L6.3mm_D2.5mm_P7.62mm_Horizontal, B.Cu at (135.0, 100.0)
- added R11: R, Resistor_THT:R_Axial_DIN0207_L6.3mm_D2.5mm_P7.62mm_Horizontal, B.Cu at (154.0, 100.0)
- added R12: R, Resistor_THT:R_Axial_DIN0207_L6.3mm_D2.5mm_P7.62mm_Horizontal, B.Cu at (173.0, 100.0)
- added R13: R, Resistor_THT:R_Axial_DIN0207_L6.3mm_D2.5mm_P7.62mm_Horizontal, B.Cu at (116.0, 119.0)
- added R14: R, Resistor_THT:R_Axial_DIN0207_L6.3mm_D2.5mm_P7.62mm_Horizontal, B.Cu at (135.0, 119.0)
- added R15: R, Resistor_THT:R_Axial_DIN0207_L6.3mm_D2.5mm_P7.62mm_Horizontal, B.Cu at (154.0, 119.0)
- added R16: R, Resistor_THT:R_Axial_DIN0207_L6.3mm_D2.5mm_P7.62mm_Horizontal, B.Cu at (173.0, 119.0)
- added R2: R, Resistor_THT:R_Axial_DIN0207_L6.3mm_D2.5mm_P7.62mm_Horizontal, B.Cu at (126.4, 62.0)
- added R3: R, Resistor_THT:R_Axial_DIN0207_L6.3mm_D2.5mm_P7.62mm_Horizontal, B.Cu at (153.0, 62.0)
- added R4: R, Resistor_THT:R_Axial_DIN0207_L6.3mm_D2.5mm_P7.62mm_Horizontal, B.Cu at (165.0, 62.0)
- added R5: R, Resistor_THT:R_Axial_DIN0207_L6.3mm_D2.5mm_P7.62mm_Horizontal, B.Cu at (116.0, 81.0)
- added R6: R, Resistor_THT:R_Axial_DIN0207_L6.3mm_D2.5mm_P7.62mm_Horizontal, B.Cu at (135.0, 81.0)
- added R7: R, Resistor_THT:R_Axial_DIN0207_L6.3mm_D2.5mm_P7.62mm_Horizontal, B.Cu at (154.0, 81.0)
- added R8: R, Resistor_THT:R_Axial_DIN0207_L6.3mm_D2.5mm_P7.62mm_Horizontal, B.Cu at (173.0, 81.0)
- added R9: R, Resistor_THT:R_Axial_DIN0207_L6.3mm_D2.5mm_P7.62mm_Horizontal, B.Cu at (116.0, 100.0)
Connections:
- net /SCL renamed SCL
- net /SDA renamed SDA
- D17 pad 2: +3V3 -> Net-(D17-A)
- D18 pad 2: +3V3 -> Net-(D18-A)
- D19 pad 2: +3V3 -> Net-(D19-A)
- D20 pad 2: +3V3 -> Net-(D20-A)
- D21 pad 2: +3V3 -> Net-(D21-A)
- D22 pad 2: +3V3 -> Net-(D22-A)
- D23 pad 2: +3V3 -> Net-(D23-A)
- D24 pad 2: +3V3 -> Net-(D24-A)
- D25 pad 2: +3V3 -> Net-(D25-A)
- D26 pad 2: +3V3 -> Net-(D26-A)
- D27 pad 2: +3V3 -> Net-(D27-A)
- D28 pad 2: +3V3 -> Net-(D28-A)
- D29 pad 2: +3V3 -> Net-(D29-A)
- D30 pad 2: +3V3 -> Net-(D30-A)
- D31 pad 2: +3V3 -> Net-(D31-A)
- D32 pad 2: +3V3 -> Net-(D32-A)
- U1 pad 7: /LED Connector 0 -> unconnected-(U1-PB08_A6_D6_TX-Pad7)
Routing:
- net +3V3: track 331.2 -> 289.7 mm
- net Net-(D32-A): track 0.00 -> 17.2 mm
- net Net-(D30-A): track 0.00 -> 17.1 mm
- net Net-(D19-A): track 0.00 -> 16.6 mm
- net Net-(D31-A): track 0.00 -> 16.3 mm
- net Net-(D28-A): track 0.00 -> 16.3 mm
- net Net-(D27-A): track 0.00 -> 16.3 mm
- net Net-(D24-A): track 0.00 -> 16.3 mm
- net Net-(D29-A): track 0.00 -> 16.3 mm
- net Net-(D22-A): track 0.00 -> 16.3 mm
- net Net-(D26-A): track 0.00 -> 16.3 mm
- net Net-(D23-A): track 0.00 -> 16.3 mm
- net Net-(D25-A): track 0.00 -> 16.2 mm
- net Net-(D17-A): track 0.00 -> 16.2 mm
- net Net-(D21-A): track 0.00 -> 16.2 mm
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